File: Kicad/Vrm/Vrm.kicad_sch (KiCad schematic)
At the start: 28 parts, among them J1 Screw_Terminal_01x05, J2 AVR-JTAG-10, J3 Screw_Terminal_01x03, J4 Screw_Terminal_01x04, Q1 FMMT458TA - SOT23, SW1 Switch, U1 STM32F091RCTx

Commit message: Final Schematic
Parts:
- added R4, R5, R6, R7: 20, symbol Device:R
- U1: renamed from U?; value LTC3638 -> LTC3631
- U2: renamed from U?; value LTC3638 -> LT1302CS8
Connections:
- net at J4.3 (Pin_3): now also R6.1; no longer U1.52 (PC11)
- net at J4.4 (Pin_4): now also R7.1; no longer U1.51 (PC10)
- net at U1.16 (PA2): now also R4.1; no longer J3.1 (Pin_1)
- net at U1.17 (PA3): now also R5.1; no longer J3.2 (Pin_2)
- new net: R7.2, U1.51 (PC10)
- new net: R6.2, U1.52 (PC11)
- new net: J3.1 (Pin_1), R4.2
- new net: J3.2 (Pin_2), R5.2
Other:
- moved on the sheet: J4
Changed lines of the file:
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@@
     (stroke (width 0) (type default) (color 0 0 0 0))
   )
-  (wire (pts (xy 125.73 118.11) (xy 127 118.11))
+  (wire (pts (xy 120.65 118.11) (xy 127 118.11))
     (stroke (width 0) (type default) (color 0 0 0 0))
   )
@@
     (stroke (width 0) (type default) (color 0 0 0 0))
   )
+  (wire (pts (xy 170.18 46.99) (xy 173.99 46.99))
+    (stroke (width 0) (type default) (color 0 0 0 0))
+  )
   (wire (pts (xy 237.49 137.16) (xy 246.38 137.16))
     (stroke (width 0) (type default) (color 0 0 0 0))
   )
+  (wire (pts (xy 128.27 113.03) (xy 129.54 113.03))
+    (stroke (width 0) (type default) (color 0 0 0 0))
+  )
   (wire (pts (xy 99.06 96.52) (xy 101.6 96.52))
     (stroke (width 0) (type default) (color 0 0 0 0))
@@
     (stroke (width 0) (type default) (color 0 0 0 0))
   )
-  (wire (pts (xy 125.73 113.03) (xy 129.54 113.03))
-    (stroke (width 0) (type default) (color 0 0 0 0))
-  )
   (wire (pts (xy 212.09 127) (xy 212.09 128.27))
     (stroke (width 0) (type default) (color 0 0 0 0))
@@
     (stroke (width 0) (type default) (color 0 0 0 0))
   )
-  (wire (pts (xy 125.73 110.49) (xy 129.54 110.49))
-    (stroke (width 0) (type default) (color 0 0 0 0))
-  )
   (wire (pts (xy 90.17 142.24) (xy 95.25 142.24))
     (stroke (width 0) (type default) (color 0 0 0 0))
@@
     (stroke (width 0) (type default) (color 0 0 0 0))
   )
+  (wire (pts (xy 170.18 49.53) (xy 173.99 49.53))
+    (stroke (width 0) (type default) (color 0 0 0 0))
+  )
   (wire (pts (xy 162.56 74.93) (xy 166.37 74.93))
     (stroke (width 0) (type default) (color 0 0 0 0))
@@
     (stroke (width 0) (type default) (color 0 0 0 0))
   )
-  (wire (pts (xy 125.73 115.57) (xy 127 115.57))
-    (stroke (width 0) (type default) (color 0 0 0 0))
-  )
   (wire (pts (xy 55.88 137.16) (xy 90.17 137.16))
     (stroke (width 0) (type default) (color 0 0 0 0))
@@
     (stroke (width 0) (type default) (color 0 0 0 0))
   )
-  (wire (pts (xy 162.56 46.99) (xy 173.99 46.99))
-    (stroke (width 0) (type default) (color 0 0 0 0))
-  )
   (wire (pts (xy 90.17 137.16) (xy 90.17 142.24))
     (stroke (width 0) (type default) (color 0 0 0 0))
@@
     (stroke (width 0) (type default) (color 0 0 0 0))
   )
-  (wire (pts (xy 162.56 49.53) (xy 173.99 49.53))
-    (stroke (width 0) (type default) (color 0 0 0 0))
-  )
   (wire (pts (xy 147.32 34.29) (xy 147.32 36.83))
     (stroke (width 0) (type default) (color 0 0 0 0))
@@
   )
   (wire (pts (xy 53.34 100.33) (xy 55.88 100.33))
+    (stroke (width 0) (type default) (color 0 0 0 0))
+  )
+  (wire (pts (xy 128.27 110.49) (xy 129.54 110.49))
     (stroke (width 0) (type default) (color 0 0 0 0))
   )
@@
   (symbol (lib_name "LTC3638_1") (lib_id "Regulator_Switching:LTC3638") (at 66.04 149.86 0) (unit 1)
     (in_bom yes) (on_board yes)
-    (property "Reference" "U?" (id 0) (at 68.58 153.67 0))
-    (property "Value" "LTC3638" (id 1) (at 68.58 156.21 0))
+    (property "Reference" "U2" (id 0) (at 68.58 153.67 0))
+    (property "Value" "LT1302CS8" (id 1) (at 68.58 156.21 0))
     (property "Footprint" "Package_SO:Linear_MSOP-12-16-1EP_3x4mm_P0.5mm" (id 2) (at 67.31 161.29 0)
       (effects (font (size 1.27 1.27)) (justify left) hide)
@@
     (pin "8")
   )
-  (symbol (lib_id "Connector:Screw_Terminal_01x04") (at 120.65 115.57 180) (unit 1)
-    (in_bom yes) (on_board yes)
-    (property "Reference" "J4" (id 0) (at 120.65 105.41 0))
-    (property "Value" "Screw_Terminal_01x04" (id 1) (at 116.84 107.95 0))
-    (property "Footprint" "" (id 2) (at 120.65 115.57 0)
-      (effects (font (size 1.27 1.27)) hide)
-    )
-    (property "Datasheet" "~" (id 3) (at 120.65 115.57 0)
+  (symbol (lib_id "Connector:Screw_Terminal_01x04") (at 115.57 115.57 180) (unit 1)
+    (in_bom yes) (on_board yes)
+    (property "Reference" "J4" (id 0) (at 115.57 107.95 0))
+    (property "Value" "Screw_Terminal_01x04" (id 1) (at 111.76 107.95 0)
+      (effects (font (size 1.27 1.27)) hide)
+    )
+    (property "Footprint" "" (id 2) (at 115.57 115.57 0)
+      (effects (font (size 1.27 1.27)) hide)
+    )
+    (property "Datasheet" "~" (id 3) (at 115.57 115.57 0)
       (effects (font (size 1.27 1.27)) hide)
     )
@@
     (pin "2")
   )
+  (symbol (lib_id "Device:R") (at 166.37 46.99 90) (unit 1)
+    (in_bom yes) (on_board yes)
+    (property "Reference" "R4" (id 0) (at 166.37 41.91 90))
+    (property "Value" "20" (id 1) (at 166.37 44.45 90))
+    (property "Footprint" "" (id 2) (at 166.37 48.768 90)
+      (effects (font (size 1.27 1.27)) hide)
+    )
+    (property "Datasheet" "~" (id 3) (at 166.37 46.99 0)
+      (effects (font (size 1.27 1.27)) hide)
+    )
+    (pin "1")
+    (pin "2")
+  )
+  (symbol (lib_id "Device:R") (at 124.46 113.03 90) (unit 1)
+    (in_bom yes) (on_board yes)
+    (property "Reference" "R6" (id 0) (at 123.19 115.57 90))
+    (property "Value" "20" (id 1) (at 127 115.57 90))
+    (property "Footprint" "" (id 2) (at 124.46 114.808 90)
+      (effects (font (size 1.27 1.27)) hide)
+    )
+    (property "Datasheet" "~" (id 3) (at 124.46 113.03 0)
+      (effects (font (size 1.27 1.27)) hide)
+    )
+    (pin "1")
+    (pin "2")
+  )
   (symbol (lib_id "dk_Transistors-Bipolar-BJT-Single:FMMT458TA") (at 219.71 62.23 0) (unit 1)
     (in_bom yes) (on_board yes) (fields_autoplaced)
@@
     (pin "2")
   )
+  (symbol (lib_id "Device:R") (at 166.37 49.53 90) (unit 1)
+    (in_bom yes) (on_board yes)
+    (property "Reference" "R5" (id 0) (at 165.1 54.61 90))
+    (property "Value" "20" (id 1) (at 165.1 52.07 90))
+    (property "Footprint" "" (id 2) (at 166.37 51.308 90)
+      (effects (font (size 1.27 1.27)) hide)
+    )
+    (property "Datasheet" "~" (id 3) (at 166.37 49.53 0)
+      (effects (font (size 1.27 1.27)) hide)
+    )
+    (pin "1")
+    (pin "2")
+  )
   (symbol (lib_name "LTC3638_1") (lib_id "Regulator_Switching:LTC3638") (at 69.85 104.14 0) (unit 1)
     (in_bom yes) (on_board yes)
-    (property "Reference" "U?" (id 0) (at 72.39 107.95 0))
-    (property "Value" "LTC3638" (id 1) (at 72.39 110.49 0))
+    (property "Reference" "U1" (id 0) (at 72.39 107.95 0))
+    (property "Value" "LTC3631" (id 1) (at 72.39 110.49 0))
     (property "Footprint" "Package_SO:Linear_MSOP-12-16-1EP_3x4mm_P0.5mm" (id 2) (at 71.12 115.57 0)
       (effects (font (size 1.27 1.27)) (justify left) hide)
@@
     (pin "2")
   )
+  (symbol (lib_id "Device:R") (at 124.46 110.49 90) (unit 1)
+    (in_bom yes) (on_board yes)
+    (property "Reference" "R7" (id 0) (at 124.46 105.41 90))
+    (property "Value" "20" (id 1) (at 124.46 107.95 90))
+    (property "Footprint" "" (id 2) (at 124.46 112.268 90)
+      (effects (font (size 1.27 1.27)) hide)
+    )
+    (property "Datasheet" "~" (id 3) (at 124.46 110.49 0)
+      (effects (font (size 1.27 1.27)) hide)
+    )
+    (pin "1")
+    (pin "2")
+  )
   (symbol (lib_id "Connector:Screw_Terminal_01x03") (at 179.07 49.53 0) (unit 1)
     (in_bom yes) (on_board yes) (fields_autoplaced)
@@
       (reference "R3") (unit 1) (value "1k") (footprint "")
     )
+    (path "/86911fa3-5320-4fab-8a10-45972c9e7dbc"
+      (reference "R4") (unit 1) (value "20") (footprint "")
+    )
     (path "/998d526c-6e7d-47fe-a455-2eae5f49a0c3"
       (reference "R4") (unit 1) (value "47k") (footprint "")
     )
+    (path "/88c7945e-cec3-40d0-b105-3941378045bb"
+      (reference "R5") (unit 1) (value "20") (footprint "")
+    )
+    (path "/86fd7e02-87e1-4ea8-9bdc-30f3b874396b"
+      (reference "R6") (unit 1) (value "20") (footprint "")
+    )
+    (path "/cdedb03e-1eac-42c8-ae28-227d4149854a"
+      (reference "R7") (unit 1) (value "20") (footprint "")
+    )
     (path "/ec4205fe-0ad3-4690-b0f4-86be32fdc5c1"
       (reference "SW1") (unit 1) (value "Switch") (footprint "")
@@
       (reference "U1") (unit 1) (value "STM32F091RCTx") (footprint "Package_QFP:LQFP-64_10x10mm_P0.5mm")
     )
+    (path "/8c5a2e91-d546-4447-a1a5-de3fc28a0599"
+      (reference "U1") (unit 1) (value "LTC3631") (footprint "Package_SO:Linear_MSOP-12-16-1EP_3x4mm_P0.5mm")
+    )
     (path "/005d4c57-73da-4414-bd13-57c3825c1db0"
-      (reference "U?") (unit 1) (value "LTC3638") (footprint "Package_SO:Linear_MSOP-12-16-1EP_3x4mm_P0.5mm")
-    )
-    (path "/8c5a2e91-d546-4447-a1a5-de3fc28a0599"
-      (reference "U?") (unit 1) (value "LTC3638") (footprint "Package_SO:Linear_MSOP-12-16-1EP_3x4mm_P0.5mm")
-    )
-  )
+      (reference "U2") (unit 1) (value "LT1302CS8") (footprint "Package_SO:Linear_MSOP-12-16-1EP_3x4mm_P0.5mm")
+    )
+  )
