File: Kicad/Vrm/Vrm.kicad_pcb (KiCad board)
At the start: 2 copper layers, 94 x 100.3 mm, 51 parts, among them U1 STM32F091RCTx

Commit message: Added Gerber file and logo
Parts:
- added 2022: LOGO, footprints:VRm_logo, F.Cu at (144.8, 132.1)
- REF** (x4): value MountingHole_3.5mm -> Mounting3.5mm
